File: electrics/scheme/voltamper.sch (KiCad schematic (older format))
At the start: 20 parts

Commit message: a
Parts:
- added C? (x2): 18p, symbol C
- added R?: 100, ~, symbol R
Connections:
- wire segments 82 -> 95
Changed lines of the file:
@@
 	1    0    0    -1
 $EndComp
+$Comp
+L GND #PWR?
+U 1 1 5480CD20
+P 1200 5700
+F 0 "#PWR?" H 1200 5700 30  0001 C CNN
+F 1 "GND" H 1200 5630 30  0001 C CNN
+F 2 "" H 1200 5700 60  0001 C CNN
+F 3 "" H 1200 5700 60  0001 C CNN
+	1    1200 5700
+	1    0    0    -1
+$EndComp
+$Comp
+L C C?
+U 1 1 5480CD26
+P 1600 6700
+F 0 "C?" H 1650 6800 50  0000 L CNN
+F 1 "18p" H 1650 6600 50  0000 L CNN
+F 2 "" H 1600 6700 60  0001 C CNN
+F 3 "" H 1600 6700 60  0001 C CNN
+	1    1600 6700
+	0    -1   -1   0
+$EndComp
+$Comp
+L C C?
+U 1 1 5480CD2C
+P 1600 5500
+F 0 "C?" H 1650 5600 50  0000 L CNN
+F 1 "18p" H 1650 5400 50  0000 L CNN
+F 2 "" H 1600 5500 60  0001 C CNN
+F 3 "" H 1600 5500 60  0001 C CNN
+	1    1600 5500
+	0    -1   -1   0
+$EndComp
+Wire Wire Line
+	2400 6500 2400 6700
+Wire Wire Line
+	1800 6700 2850 6700
+Wire Wire Line
+	2000 5700 2000 5500
+Wire Wire Line
+	1800 5500 3700 5500
+Wire Wire Line
+	1400 5500 1200 5500
+Wire Wire Line
+	1200 5500 1200 5700
+Wire Wire Line
+	1400 6700 1200 6700
+Wire Wire Line
+	1200 6700 1200 6900
+$Comp
+L GND #PWR?
+U 1 1 5480CD40
+P 1200 6900
+F 0 "#PWR?" H 1200 6900 30  0001 C CNN
+F 1 "GND" H 1200 6830 30  0001 C CNN
+F 2 "" H 1200 6900 60  0001 C CNN
+F 3 "" H 1200 6900 60  0001 C CNN
+	1    1200 6900
+	1    0    0    -1
+$EndComp
+Connection ~ 2000 5500
+Connection ~ 2400 6700
+$Comp
+L R R?
+U 1 1 5480CD4A
+P 3100 6700
+F 0 "R?" V 3180 6700 40  0000 C CNN
+F 1 "100" V 3107 6701 40  0000 C CNN
+F 2 "~" V 3030 6700 30  0000 C CNN
+F 3 "~" H 3100 6700 30  0000 C CNN
+	1    3100 6700
+	0    -1   -1   0
+$EndComp
+Wire Wire Line
+	2400 5700 2400 5650
+Wire Wire Line
+	2400 5650 2600 5650
+Wire Wire Line
+	2600 5650 2600 5750
+$Comp
+L GND #PWR?
+U 1 1 5480CD54
+P 2600 5750
+F 0 "#PWR?" H 2600 5750 30  0001 C CNN
+F 1 "GND" H 2600 5680 30  0001 C CNN
+F 2 "" H 2600 5750 60  0001 C CNN
+F 3 "" H 2600 5750 60  0001 C CNN
+	1    2600 5750
+	1    0    0    -1
+$EndComp
+Wire Wire Line
+	2000 6500 2000 6600
+$Comp
+L GND #PWR?
+U 1 1 5480CD5B
+P 2000 6600
+F 0 "#PWR?" H 2000 6600 30  0001 C CNN
+F 1 "GND" H 2000 6530 30  0001 C CNN
+F 2 "" H 2000 6600 60  0001 C CNN
+F 3 "" H 2000 6600 60  0001 C CNN
+	1    2000 6600
+	1    0    0    -1
+$EndComp
+Wire Wire Line
+	3350 6700 3700 6700
 $EndSCHEMATC

Commit message: a
Parts:
- added C?: 100u, ~, symbol CP1
- added C?: 10u, symbol C
- added D?: DIODE, ~, symbol DIODE
- added U?: CRYSTAL-4PIN, ~, symbol CRYSTAL-4PIN
- added U?: MCP1703T-3302E/CB, ~, symbol MCP1703T-3302E/CB
Connections:
- net labels added: Vbus, Vin
- wire segments 95 -> 114
Other:
- moved on the sheet: C?
Changed lines of the file:
@@
 LIBS:cp2102
 LIBS:micro-usb-b
+LIBS:crystal-4pin
+LIBS:mcp1703t-3302e
+LIBS:ncp3063
 LIBS:voltamper-cache
 EELAYER 27 0
@@
 Sheet 1 1
 Title ""
-Date "4 dec 2014"
+Date "5 dec 2014"
 Rev ""
 Comp ""
@@
 	20050 5350 20050 5400
 Wire Wire Line
-	20400 4950 20050 4950
-Wire Wire Line
-	20050 4950 20050 4600
+	20050 4950 20400 4950
+Wire Wire Line
+	20050 4300 20050 4950
 $Comp
 L R R?
@@
 L GND #PWR?
 U 1 1 5480CD20
-P 1200 5700
-F 0 "#PWR?" H 1200 5700 30  0001 C CNN
-F 1 "GND" H 1200 5630 30  0001 C CNN
-F 2 "" H 1200 5700 60  0001 C CNN
-F 3 "" H 1200 5700 60  0001 C CNN
-	1    1200 5700
+P 1200 5100
+F 0 "#PWR?" H 1200 5100 30  0001 C CNN
+F 1 "GND" H 1200 5030 30  0001 C CNN
+F 2 "" H 1200 5100 60  0001 C CNN
+F 3 "" H 1200 5100 60  0001 C CNN
+	1    1200 5100
 	1    0    0    -1
 $EndComp
@@
 L C C?
 U 1 1 5480CD2C
-P 1600 5500
-F 0 "C?" H 1650 5600 50  0000 L CNN
-F 1 "18p" H 1650 5400 50  0000 L CNN
-F 2 "" H 1600 5500 60  0001 C CNN
-F 3 "" H 1600 5500 60  0001 C CNN
-	1    1600 5500
+P 1600 4900
+F 0 "C?" H 1650 5000 50  0000 L CNN
+F 1 "18p" H 1650 4800 50  0000 L CNN
+F 2 "" H 1600 4900 60  0001 C CNN
+F 3 "" H 1600 4900 60  0001 C CNN
+	1    1600 4900
 	0    -1   -1   0
 $EndComp
@@
 	1800 6700 2850 6700
 Wire Wire Line
-	2000 5700 2000 5500
-Wire Wire Line
-	1800 5500 3700 5500
-Wire Wire Line
-	1400 5500 1200 5500
-Wire Wire Line
-	1200 5500 1200 5700
+	2000 5100 2000 4900
+Wire Wire Line
+	1400 4900 1200 4900
+Wire Wire Line
+	1200 4900 1200 5100
 Wire Wire Line
 	1400 6700 1200 6700
@@
 	1    0    0    -1
 $EndComp
-Connection ~ 2000 5500
+Connection ~ 2000 4900
 Connection ~ 2400 6700
 $Comp
@@
 $EndComp
 Wire Wire Line
-	2400 5700 2400 5650
-Wire Wire Line
-	2400 5650 2600 5650
-Wire Wire Line
-	2600 5650 2600 5750
+	2400 5100 2400 5050
+Wire Wire Line
+	2400 5050 2600 5050
+Wire Wire Line
+	2600 5050 2600 5150
 $Comp
 L GND #PWR?
 U 1 1 5480CD54
-P 2600 5750
-F 0 "#PWR?" H 2600 5750 30  0001 C CNN
-F 1 "GND" H 2600 5680 30  0001 C CNN
-F 2 "" H 2600 5750 60  0001 C CNN
-F 3 "" H 2600 5750 60  0001 C CNN
-	1    2600 5750
+P 2600 5150
+F 0 "#PWR?" H 2600 5150 30  0001 C CNN
+F 1 "GND" H 2600 5080 30  0001 C CNN
+F 2 "" H 2600 5150 60  0001 C CNN
+F 3 "" H 2600 5150 60  0001 C CNN
+	1    2600 5150
 	1    0    0    -1
 $EndComp
@@
 Wire Wire Line
 	3350 6700 3700 6700
+$Comp
+L CRYSTAL-4PIN U?
+U 1 1 54812E0A
+P 2200 5800
+F 0 "U?" H 2200 5500 60  0000 C CNN
+F 1 "CRYSTAL-4PIN" H 2200 6150 60  0000 C CNN
+F 2 "~" H 2150 5800 60  0000 C CNN
+F 3 "~" H 2150 5800 60  0000 C CNN
+	1    2200 5800
+	0    1    1    0
+$EndComp
+Wire Wire Line
+	3700 5500 3100 5500
+Wire Wire Line
+	3100 5500 3100 4900
+Wire Wire Line
+	3100 4900 1800 4900
+$Comp
+L MCP1703T-3302E/CB U?
+U 1 1 548149DE
+P 12250 1900
+F 0 "U?" H 12250 1850 60  0000 C CNN
+F 1 "MCP1703T-3302E/CB" H 12250 2200 60  0000 C CNN
+F 2 "~" H 12250 1900 60  0000 C CNN
+F 3 "~" H 12250 1900 60  0000 C CNN
+	1    12250 1900
+	1    0    0    -1
+$EndComp
+Wire Wire Line
+	12250 2550 12250 2750
+$Comp
+L GND #PWR?
+U 1 1 548149E5
+P 12250 2750
+F 0 "#PWR?" H 12250 2750 30  0001 C CNN
+F 1 "GND" H 12250 2680 30  0001 C CNN
+F 2 "" H 12250 2750 60  0000 C CNN
+F 3 "" H 12250 2750 60  0000 C CNN
+	1    12250 2750
+	1    0    0    -1
+$EndComp
+$Comp
+L DIODE D?
+U 1 1 548149EB
+P 11100 1800
+F 0 "D?" H 11100 1900 40  0000 C CNN
+F 1 "DIODE" H 11100 1700 40  0000 C CNN
+F 2 "~" H 11100 1800 60  0000 C CNN
+F 3 "~" H 11100 1800 60  0000 C CNN
+	1    11100 1800
+	1    0    0    -1
+$EndComp
+Wire Wire Line
+	11300 1800 11700 1800
+Wire Wire Line
+	11500 1000 11500 2000
+Connection ~ 11500 1800
+$Comp
+L CP1 C?
+U 1 1 548149F4
+P 11500 2200
+F 0 "C?" H 11550 2300 50  0000 L CNN
+F 1 "100u" H 11550 2100 50  0000 L CNN
+F 2 "~" H 11500 2200 60  0000 C CNN
+F 3 "~" H 11500 2200 60  0000 C CNN
+	1    11500 2200
+	1    0    0    -1
+$EndComp
+Wire Wire Line
+	11500 2400 11500 2600
+$Comp
+L GND #PWR?
+U 1 1 548149FB
+P 11500 2600
+F 0 "#PWR?" H 11500 2600 30  0001 C CNN
+F 1 "GND" H 11500 2530 30  0001 C CNN
+F 2 "" H 11500 2600 60  0000 C CNN
+F 3 "" H 11500 2600 60  0000 C CNN
+	1    11500 2600
+	1    0    0    -1
+$EndComp
+Wire Wire Line
+	12800 1800 13000 1800
+Wire Wire Line
+	13000 1600 13000 2000
+$Comp
+L VDD #PWR?
+U 1 1 54814A03
+P 13000 1600
+F 0 "#PWR?" H 13000 1700 30  0001 C CNN
+F 1 "VDD" H 13000 1710 30  0000 C CNN
+F 2 "" H 13000 1600 60  0001 C CNN
+F 3 "" H 13000 1600 60  0001 C CNN
+	1    13000 1600
+	1    0    0    -1
+$EndComp
+Wire Wire Line
+	10900 1800 10700 1800
+Text Label 10700 1750 1    60   ~ 0
+Vbus
+Wire Wire Line
+	10700 1800 10700 1600
+Wire Wire Line
+	10700 1200 10700 1000
+Text Label 10700 1150 1    60   ~ 0
+Vin
+Connection ~ 13000 1800
+$Comp
+L C C?
+U 1 1 54814A15
+P 13000 2200
+F 0 "C?" H 13050 2300 50  0000 L CNN
+F 1 "10u" H 13050 2100 50  0000 L CNN
+F 2 "" H 13000 2200 60  0001 C CNN
+F 3 "" H 13000 2200 60  0001 C CNN
+	1    13000 2200
+	1    0    0    -1
+$EndComp
+Wire Wire Line
+	10700 1200 11500 1200
+Wire Wire Line
+	13000 2400 13000 2600
+$Comp
+L GND #PWR?
+U 1 1 54814A1E
+P 13000 2600
+F 0 "#PWR?" H 13000 2600 30  0001 C CNN
+F 1 "GND" H 13000 2530 30  0001 C CNN
+F 2 "" H 13000 2600 60  0000 C CNN
+F 3 "" H 13000 2600 60  0000 C CNN
+	1    13000 2600
+	1    0    0    -1
+$EndComp
+$Comp
+L PWR_FLAG #FLG?
+U 1 1 54814A24
+P 11500 1000
+F 0 "#FLG?" H 11500 1095 30  0001 C CNN
+F 1 "PWR_FLAG" H 11500 1180 30  0000 C CNN
+F 2 "" H 11500 1000 60  0000 C CNN
+F 3 "" H 11500 1000 60  0000 C CNN
+	1    11500 1000
+	1    0    0    -1
+$EndComp
+Connection ~ 11500 1200
+Connection ~ 20050 4600
+Text Label 20050 4500 1    60   ~ 0
+Vbus
+Wire Wire Line
+	4700 13450 4700 13750
+Wire Wire Line
+	4700 13750 5800 13750
+Wire Wire Line
+	5800 13750 5800 13450
+Wire Wire Line
+	5600 13450 5600 13750
+Connection ~ 5600 13750
+Wire Wire Line
+	5400 13450 5400 13750
+Connection ~ 5400 13750
+Wire Wire Line
+	5200 13450 5200 13750
+Connection ~ 5200 13750
 $EndSCHEMATC

Commit message: a
Parts:
- added C?: 1u, ~, symbol C
- added C?: 10u, symbol C
- added D?: AD8607, symbol AD8607
- added R?: 10, ~, symbol R
- added R?: 80k, ~, symbol R
- added R? (x3): R, ~, symbol R
- added U?: INA126, symbol INA126
- added U?: TDA2030A, ~, symbol TDA2030A
- added U?: MCP1703T-3302E/CB, ~, symbol MCP1703T-3302E/CB
Connections:
- net labels added: v+, v-
- wire segments 114 -> 142
Other:
- moved on the sheet: C?, D?

Commit message: a
Parts:
- added C? (x3): 10n, ~, symbol C
- added C?: 100n, ~, symbol C
- added D?: AD8607, symbol AD8607
- added R? (x2): 20k, ~, symbol R
- added R?: 100, ~, symbol R
- added R?: 10k, ~, symbol R
- added R? (x2): 1k, ~, symbol R
- added R?: 10, ~, symbol R
- added R?: R, ~, symbol R
- added U?: TDA2030A, ~, symbol TDA2030A
- C? (x2): value 10u -> 4u7
- R?: value R -> 10k
Connections:
- net labels added: AVdd, Eprobe, Eref, Esen, dac-high, dac-low
- wire segments 142 -> 193
Other:
- note added: "G=5+80k/Rg"
- note added: "Vin=0..Vpp => Vout=-2Vpp..2Vpp"
- moved on the sheet: C?, D?, R?, U?

Commit message: a
Other:
- note added: "Here it's wrong as it is impossible to \nmake low-dac to be in the middle of the range."
- moved on the sheet: C?, D?, R?, U?

Commit message: a
Parts:
- removed C?: 100n, ~, symbol C
- removed C? (x2): 10n, ~, symbol C
- removed R? (x2): R, ~, symbol R
- removed R?: 100, ~, symbol R
- removed R?: 10k, ~, symbol R
- removed R?: 10, ~, symbol R
- removed U?: TDA2030A, ~, symbol TDA2030A
- added C?: 10n, ~, symbol C
- added R? (x3): R, ~, symbol R
- R?: value 80k -> 16k
- R?: value R -> 10k
- R?: value 1k -> 33k
Connections:
- net labels added: Eaux, Eaux-test, Ework, VPP, Vpp-in
- net labels removed: Eprobe, Esen
- wire segments 193 -> 175
Other:
- note added: "-2Vpp..2Vpp"
- note added: "G=10 if Rg=16k"
- note added: "I +/-50mA => +/-0.5V (G=10) =>+/-5V"
- note added: "V+/-5V"
- note removed: "Here it's wrong as it is impossible to \nmake low-dac to be in the middle of the range."

Commit message: a
Parts:
- removed C?: 4u7, ~, symbol C
- removed C?: 10n, ~, symbol C
- removed L?: INDUCTOR_SMALL, ~, symbol INDUCTOR_SMALL
- removed R?: 10k, ~, symbol R
- removed R?: R, ~, symbol R
- added R? (x4): R, ~, symbol R
- added R? (x4): 10k, ~, symbol R
Connections:
- net labels added: Eaux-in, Eref-in, Eref-test, Iref, Iref-in, Vpp/2
- net labels removed: Vpp-in
- wire segments 175 -> 193
Other:
- moved on the sheet: C?, D?, R?, U?

Commit message: a
Parts:
- added C?: 100n, ~, symbol C
- added C? (x2): CP, ~, symbol CP
- added C?: 2n2, ~, symbol C
- added C?: C, ~, symbol C
- added D?: DIODESCH, ~, symbol DIODESCH
- added D?: DIODE, ~, symbol DIODE
- added L?: 50uH, ~, symbol INDUCTOR_SMALL
- added R?: 0.25, ~, symbol R
- added R?: 1k1, ~, symbol R
- added R?: 10k, ~, symbol R
- added U?: NCP3063, ~, symbol NCP3063
Connections:
- net labels added: +, -
- wire segments 193 -> 225
Other:
- moved on the sheet: C?, R?, U?
