File: electrics/scheme/voltamper.sch (KiCad schematic (older format))
At the start: 63 parts

Commit message: a
Parts:
- removed C? (x2): CP, ~, symbol CP
- removed R? (x3): 10k, ~, symbol R
- added C? (x4): 100n, ~, symbol C
- added C?: 2n2, ~, symbol C
- added C? (x2): C, ~, symbol C
- added C? (x3): 330u, ~, symbol CP1
- added D?: 1N5819, ~, symbol DIODESCH
- added L?: 30uH, ~, symbol INDUCTOR_SMALL
- added R?: 0.15, ~, symbol R
- added R?: 1k1, ~, symbol R
- added R?: 10k, ~, symbol R
- added R? (x3): 1k33, ~, symbol R
- added R?: 1k, ~, symbol R
- added U?: NCP3063, ~, symbol NCP3063
- D?: value DIODESCH -> 1N5819
- R?: value 16k -> 5.3
- R?: value 20k -> 1k
- R?: value 20k -> 6k8
- R? (x3): value R -> 1k
- R? (x3): value R -> 4k
- R?: value 0.25 -> 0.15
Connections:
- wire segments 225 -> 262
Other:
- note added: "-11.7..+11.7"
- note added: "Rg=6.8 => G=1+80/6.8 = 12.76"
- note added: "V = +/-10V"
- note added: "Vin=0..3V => Vout=-11.7V..11.7V"
- note removed: "-2Vpp..2Vpp"
- note removed: "G=10 if Rg=16k"
- note removed: "V+/-5V"
- note removed: "Vin=0..Vpp => Vout=-2Vpp..2Vpp"
- moved on the sheet: C?, D?, R?

Commit message: a
Parts:
- added K?: servo-1, symbol CONN_3
- added K?: servo-2, symbol CONN_3
- added Q?: irlml2244, ~, symbol MOSFET_P
- added Q? (x2): bc857, ~, symbol PNP
- added Q? (x2): bc847, ~, symbol NPN
- added R? (x2): 3, ~, symbol R
- added R? (x2): 30k, ~, symbol R
- added R? (x2): 1k, ~, symbol R
- added R?: 10, ~, symbol R
- added R? (x2): 100, ~, symbol R
- C?: value C -> 10n
Connections:
- net labels added: gate, servo-1-pwm, servo-2-pwm, servo-en-400mA, servo-en-60mA, servo-vcc, src
- wire segments 262 -> 301

Commit message: a
Parts:
- added P?: aux, ~, symbol TST
- added P?: ref, ~, symbol TST
- added P?: work, ~, symbol TST
- added P?: +, ~, symbol TST
- added P?: -, ~, symbol TST
- added P? (x2): boot, symbol CONN_2
- added Q? (x3): NPN, ~, symbol NPN
- added R? (x4): 1k, ~, symbol R
- added R?: 10k, symbol R
- added U? (x3): SPARTAN-SIP-9007, ~, symbol SPARTAN-SIP-9007
- D? (x2): value DIODE -> 1N5819
Connections:
- net labels added: aux-1, aux-2, curr-1, curr-2, curr-en, eux-en, volt-1, volt-2, volt-en
- wire segments 301 -> 340
Other:
- note added: "This resistor protects two (voltage and current) \ninputs from short circuit when both relays are on."

Commit message: a
Parts:
- added R?: 10k, symbol R
Connections:
- wire segments 340 -> 343
Changed lines of the file:
@@
 	1    0    0    -1
 $EndComp
+Wire Wire Line
+	3700 12100 3500 12100
+Wire Wire Line
+	3500 12100 3500 12300
+$Comp
+L R R?
+U 1 1 54862FA8
+P 3500 12550
+F 0 "R?" V 3580 12550 50  0000 C CNN
+F 1 "10k" V 3500 12550 50  0000 C CNN
+F 2 "" H 3500 12550 60  0001 C CNN
+F 3 "" H 3500 12550 60  0001 C CNN
+	1    3500 12550
+	1    0    0    -1
+$EndComp
+$Comp
+L GND #PWR?
+U 1 1 54862FAE
+P 3500 13000
+F 0 "#PWR?" H 3500 13000 30  0001 C CNN
+F 1 "GND" H 3500 12930 30  0001 C CNN
+F 2 "" H 3500 13000 60  0001 C CNN
+F 3 "" H 3500 13000 60  0001 C CNN
+	1    3500 13000
+	1    0    0    -1
+$EndComp
+Wire Wire Line
+	3500 12800 3500 13000
 $EndSCHEMATC

Commit message: a
Parts:
- added C? (x9): 100n, ~, symbol C
- added C?: 10n, ~, symbol C
- added K?: swd, symbol CONN_3
Connections:
- net labels added: aux-en, swd-clk, swd-io
- net labels removed: eux-en
- wire segments 343 -> 392
- no-connect marks 7 -> 38
Other:
- moved on the sheet: P?

Commit message: a
Other:
- note added: "Here opamps in 1:1 mode because later voltage \nis mixed using resistor voltage divider. And \nbecause of this it needs isolation."
Changed lines of the file:
@@
 	9550 1150 9550 1000
 Connection ~ 10000 1150
+Text Notes 29400 19700 0    60   ~ 0
+Here opamps in 1:1 mode because later voltage \nis mixed using resistor voltage divider. And \nbecause of this it needs isolation.
 $EndSCHEMATC

Commit message: a
Parts:
- C15: renamed from C?; value 100u -> 330u
- C4: renamed from C?; value C -> 100n
- D4, D6: renamed from D?; value AD8607 -> lm258a
- L2: renamed from L?; value 30uH -> 50uH
- Q6, Q7, Q8: renamed from Q?; value NPN -> bc847
- R15, R9: renamed from R?; value 30k -> 10k
- R21: renamed from R?; value 33k -> 30k
- R4: renamed from R?; value R -> 10k
- R40: renamed from R?; value 5.3 -> 5k3
- gave numbers to parts that had none: 111
Connections:
- net labels removed: VPP
- wire segments 392 -> 395

Commit message: a
Parts:
- added D7, D8, D9: 1N5819, ~, symbol DIODESCH
Connections:
- wire segments 395 -> 401
Changed lines of the file:
@@
 	1    0    0    -1
 $EndComp
+$Comp
+L DIODESCH D7
+U 1 1 5485E30E
+P 18700 16100
+F 0 "D7" H 18700 16200 40  0000 C CNN
+F 1 "1N5819" H 18700 16000 40  0000 C CNN
+F 2 "~" H 18700 16100 60  0000 C CNN
+F 3 "~" H 18700 16100 60  0000 C CNN
+	1    18700 16100
+	0    -1   -1   0
+$EndComp
+Wire Wire Line
+	18700 15900 18500 15900
+Connection ~ 18500 15900
+Wire Wire Line
+	18700 16300 18500 16300
+Connection ~ 18500 16300
+$Comp
+L DIODESCH D8
+U 1 1 5485E6E8
+P 20500 16100
+F 0 "D8" H 20500 16200 40  0000 C CNN
+F 1 "1N5819" H 20500 16000 40  0000 C CNN
+F 2 "~" H 20500 16100 60  0000 C CNN
+F 3 "~" H 20500 16100 60  0000 C CNN
+	1    20500 16100
+	0    -1   -1   0
+$EndComp
+Wire Wire Line
+	20500 15900 20300 15900
+Connection ~ 20300 15900
+Wire Wire Line
+	20500 16300 20300 16300
+Connection ~ 20300 16300
+$Comp
+L DIODESCH D9
+U 1 1 5485EACA
+P 22250 16100
+F 0 "D9" H 22250 16200 40  0000 C CNN
+F 1 "1N5819" H 22250 16000 40  0000 C CNN
+F 2 "~" H 22250 16100 60  0000 C CNN
+F 3 "~" H 22250 16100 60  0000 C CNN
+	1    22250 16100
+	0    -1   -1   0
+$EndComp
+Wire Wire Line
+	22250 15900 22050 15900
+Connection ~ 22050 15900
+Wire Wire Line
+	22250 16300 22050 16300
+Connection ~ 22050 16300
 $EndSCHEMATC
