File: electrics/scheme/voltamper.kicad_pcb (KiCad board)
At the start: 2 copper layers, 127 parts, among them K1 swd, K2 servo-1, K3 servo-2, P1 boot, P2 boot, P3 -, P4 +, P5 work, P6 aux, P7 ref, Q1 bc857, Q2 bc847, Q3 bc857, Q4 bc847, Q5 irlml2244, Q6 bc847, Q7 bc847, Q8 bc847, U1 CRYSTAL-4PIN, U10 TDA2030A, U11 INA126, U12 SPARTAN-SIP-9007, U2 CP2102, U3 MICRO-USB-B, U4 MCP1703T-3302E/CB, U5 MCP1703T-3302E/CB, U6 NCP3063, U7 SPARTAN-SIP-9007, U8 NCP3063, U9 SPARTAN-SIP-9007

Commit message: a
Parts:
- C29, C33, C40: value 100n -> 30n
Changed lines of the file:
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@@
     (links 284)
     (no_connects 284)
-    (area 0 0 0 0)
+    (area -62.9485 -48.468256 54.103888 33.215001)
     (thickness 1.6)
     (drawings 0)
@@
     (pad_to_mask_clearance 0)
     (aux_axis_origin 0 0)
-    (visible_elements FFFFFFBF)
+    (visible_elements 7FFFFFFF)
     (pcbplotparams
       (layerselection 3178497)
@@
       (effects (font (size 0.50038 0.50038) (thickness 0.10922)))
     )
-    (fp_text value 100n (at 0 0.381) (layer F.SilkS)
+    (fp_text value 30n (at 0 0.381) (layer F.SilkS)
       (effects (font (size 0.50038 0.50038) (thickness 0.10922)))
     )
@@
       (effects (font (size 0.50038 0.50038) (thickness 0.10922)))
     )
-    (fp_text value 100n (at 0 0.381) (layer F.SilkS)
+    (fp_text value 30n (at 0 0.381) (layer F.SilkS)
       (effects (font (size 0.50038 0.50038) (thickness 0.10922)))
     )
@@
       (effects (font (size 0.50038 0.50038) (thickness 0.10922)))
     )
-    (fp_text value 100n (at 0 0.381) (layer F.SilkS)
+    (fp_text value 30n (at 0 0.381) (layer F.SilkS)
       (effects (font (size 0.50038 0.50038) (thickness 0.10922)))
     )

Commit message: a
Parts:
- added D10: led-0, LED-3MM, F.Cu at (34.3, -28.0)
- added D11: led-1, LED-3MM, F.Cu at (33.9, -33.3)
- added D12: led-2, LED-3MM, F.Cu at (44.2, -32.5)
- added R44: 1k, SM0805, F.Cu at (5.00, -7.20)
- added R45: 1k, SM0805, F.Cu at (-0.10, -1.70)
- added R46: 1k, SM0805, F.Cu at (3.20, -1.70)
- added R47: 10k, SM0805, F.Cu at (-1.30, 5.10)
- added R48: 10k, SM0805, F.Cu at (-1.40, 0.80)
- added SW1: btn-1, PIN_ARRAY_2X1, F.Cu at (36.0, -22.5)
- added SW2: btn-2, PIN_ARRAY_2X1, F.Cu at (44.9, -39.5)
- moved U1 308.3 mm to (219.0, 158.7)
- moved R4 282.9 mm to (227.3, 159.1), turned to 90 degrees
- moved C3 280.9 mm to (223.4, 158.7), turned to 90 degrees
- moved C4 280.3 mm to (225.4, 159.1), turned to 270 degrees
- moved R3 279.4 mm to (222.1, 155.6), turned to 180 degrees
- moved C2 276.4 mm to (214.5, 158.7), turned to 270 degrees
- moved MCU1 262.3 mm to (221.8, 144.5)
- moved U2 256.3 mm to (221.2, 129.2)
Connections:
- MCU1 pad 26: (no net) -> /led-0
- MCU1 pad 27: (no net) -> /led-1
- MCU1 pad 29: (no net) -> /led-2
- MCU1 pad 30: (no net) -> /btn-1
- MCU1 pad 33: (no net) -> /btn-2

Commit message: a
Parts:
- removed C10: 100n, SM0805
- removed C12: 1u, SM0805
- moved D2 313.4 mm to (227.6, 117.6), turned to 270 degrees
- moved C15 298.8 mm to (241.1, 119.1), turned to 270 degrees
- moved C17 295.0 mm to (232.4, 157.4)
- moved K1 290.8 mm to (204.1, 137.2), turned to 270 degrees
- moved P2 290.1 mm to (225.5, 169.6), turned to 180 degrees
- moved C5 282.7 mm to (224.9, 156.9), turned to 270 degrees
- moved C11 276.4 mm to (230.3, 148.8), turned to 270 degrees
- moved C14 274.3 mm to (228.4, 137.3), turned to 90 degrees
- moved C7 271.8 mm to (230.4, 137.3), turned to 90 degrees
- moved U5 270.6 mm to (232.4, 160.3), turned to 180 degrees
- moved C16 269.8 mm to (233.4, 120.4), turned to 180 degrees
- moved C9 264.6 mm to (215.6, 151.3), turned to 270 degrees
- moved C13 258.9 mm to (214.9, 138.0), turned to 180 degrees
- moved C1 257.0 mm to (218.7, 130.6), turned to 180 degrees
- moved R1 256.3 mm to (218.7, 128.7)
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
Commit message: a
Parts:
- added C10: 4u7, SM0805, F.Cu at (0.00, 0.00)
Connections:
- U2 pad 10: N-0000094 -> VDD
- U2 pad 13: N-0000094 -> VDD
- U2 pad 14: N-0000094 -> VDD
- U2 pad 15: N-0000094 -> VDD
- U2 pad 16: N-0000094 -> VDD
- U2 pad 17: N-0000094 -> VDD
- U2 pad 18: N-0000094 -> N-0000061
- U2 pad 19: N-0000094 -> VDD
- U2 pad 20: N-0000094 -> VDD
- U2 pad 21: N-0000094 -> VDD
- U2 pad 22: N-0000094 -> VDD

Commit message: a
Parts:
- U2: footprint QFN28 -> CP2102

Commit message: a
Parts:
- moved D1 303.8 mm to (230.3, 117.6), turned to 270 degrees
- moved R5 289.4 mm to (233.5, 142.8)
- moved R2 276.4 mm to (203.9, 149.2), turned to 180 degrees
- moved P1 267.4 mm to (203.8, 146.5)
- moved D3 227.3 mm to (104.0, 144.4), turned to 270 degrees
- moved R29 212.1 mm to (159.6, 50.7), turned to 270 degrees
- moved D5 209.1 mm to (161.8, 60.2)
- moved C32 207.9 mm to (161.9, 52.5), turned to 90 degrees
- moved U6 199.2 mm to (102.8, 133.6)
- moved C28 196.7 mm to (158.9, 47.0)
- moved C36 195.4 mm to (172.8, 61.8), turned to 270 degrees
- moved C24 195.2 mm to (94.8, 143.9), turned to 90 degrees
- moved R28 194.4 mm to (155.3, 47.0)
- moved C18 192.3 mm to (113.7, 133.8), turned to 270 degrees
- moved R16 188.0 mm to (107.6, 142.8), turned to 270 degrees
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
Commit message: a
Parts:
- moved D7 155.5 mm to (59.3, 105.9), turned to 180 degrees
- moved D8 149.8 mm to (59.2, 90.7), turned to 180 degrees
- moved C39 148.2 mm to (82.9, 84.4), turned to 180 degrees
- moved D6 146.0 mm to (81.0, 88.5), turned to 90 degrees
- moved C42 143.8 mm to (79.3, 92.5)
- moved R19 142.6 mm to (59.2, 110.0)
- moved R35 141.7 mm to (84.0, 93.3), turned to 90 degrees
- moved Q8 130.6 mm to (42.9, 75.5), turned to 270 degrees
- moved C35 129.7 mm to (36.3, 103.2), turned to 270 degrees
- moved R26 128.7 mm to (58.3, 86.5)
- moved Q6 114.8 mm to (63.1, 109.0), turned to 180 degrees
- moved C37 114.5 mm to (38.9, 103.2), turned to 270 degrees
- moved R27 111.6 mm to (46.9, 76.3), turned to 180 degrees
- moved U9 111.5 mm to (59.4, 95.1)
- moved R40 109.3 mm to (29.1, 100.5)
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Connections:
- C22 pad 1: /aux-2 -> /v+
- C24 pad 1: /aux-2 -> /v+
- C26 pad 1: /aux-2 -> /v+
- C34 pad 1: /aux-2 -> /v+
- C35 pad 1: /aux-2 -> /v+
- C42 pad 1: /aux-2 -> /v+
- D3 pad 2: /aux-2 -> /v+
- D4 pad 8: /aux-2 -> /v+
- D6 pad 8: /aux-2 -> /v+
- D7 pad 2: /aux-2 -> /v+
- D8 pad 2: /aux-2 -> /v+
- D9 pad 2: /aux-2 -> /v+
- R16 pad 2: /aux-2 -> /v+
- U10 pad 5: /aux-2 -> /v+
- U11 pad 7: /aux-2 -> /v+
- U12 pad 3: /aux-2 -> /v+
- U7 pad 2: /aux-2 -> /v+
- U9 pad 2: /curr-1 -> /v+
- U9 pad 3: /aux-2 -> /curr-1

Commit message: a
Parts:
- moved K2 319.9 mm to (156.6, 216.7), turned to 270 degrees
- moved P3 297.4 mm to (240.2, 110.3)
- moved K3 287.5 mm to (156.6, 202.7), turned to 270 degrees
- moved R23 285.9 mm to (153.3, 214.1), turned to 180 degrees
- moved P4 283.1 mm to (233.6, 110.3)
- moved R24 275.0 mm to (153.2, 200.2)
- moved Q5 273.0 mm to (129.3, 201.7), turned to 90 degrees
- moved R10 259.9 mm to (119.0, 199.9), turned to 90 degrees
- moved C10 258.9 mm to (226.8, 124.9), turned to 270 degrees
- moved R15 251.7 mm to (123.7, 196.1)
- moved R9 248.9 mm to (123.4, 204.6)
- moved R8 247.7 mm to (117.2, 204.6), turned to 270 degrees
- moved R11 245.5 mm to (120.9, 199.9), turned to 90 degrees
- moved R7 243.8 mm to (120.0, 208.5), turned to 90 degrees
- moved R12 242.5 mm to (117.3, 196.2), turned to 270 degrees
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