File: electrics/scheme/voltamper.kicad_pcb (KiCad board)
At the start: 2 copper layers, 136 parts, among them K1 swd, K2 servo-1, K3 servo-2, P1 boot, P2 boot, P3 -, P4 +, P5 work, P6 aux, P7 ref, Q1 bc857, Q2 bc847, Q3 bc857, Q4 bc847, Q5 irlml2244, Q6 bc847, Q7 bc847, Q8 bc847, SW1 btn-1, SW2 btn-2, U1 CRYSTAL-4PIN, U10 TDA2030A, U11 INA126, U12 SPARTAN-SIP-9007, U2 CP2102, U3 MICRO-USB-B, U4 MCP1703T-3302E/CB, U5 MCP1703T-3302E/CB, U6 NCP3063, U7 SPARTAN-SIP-9007, U8 NCP3063, U9 SPARTAN-SIP-9007

Commit message: a
Parts:
- moved R48 118.7 mm to (190.8, 99.1)
- moved SW2 118.7 mm to (190.8, 94.4)
- moved D12 118.7 mm to (197.7, 94.6)
- moved R46 118.7 mm to (197.7, 99.1)
- moved D10 118.7 mm to (210.1, 94.6)
- moved D11 118.7 mm to (203.4, 94.6)
- moved R44 118.7 mm to (210.1, 99.1)
- moved R45 118.7 mm to (203.4, 99.1)
- moved R47 118.7 mm to (185.5, 99.1)
- moved SW1 118.7 mm to (185.5, 94.3)
- moved C19 108.9 mm to (214.8, 119.6)
- moved C24 108.9 mm to (202.8, 129.9)
- moved L1 108.9 mm to (203.3, 119.6)
- moved R13 108.9 mm to (210.8, 114.8)
- moved U6 108.9 mm to (210.8, 119.6)
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
Commit message: a
Parts:
- removed C18: 330u, C2V10
- moved P5 222.3 mm to (226.6, 186.4)
- moved P6 192.5 mm to (210.2, 186.5), turned to 180 degrees
- moved U12 184.8 mm to (202.7, 180.3)
- moved R39 183.1 mm to (201.2, 172.5), turned to 270 degrees
- moved D9 181.8 mm to (193.0, 184.9)
- moved Q8 180.1 mm to (185.9, 184.9), turned to 90 degrees
- moved C38 179.6 mm to (199.2, 172.5), turned to 270 degrees
- moved P7 176.6 mm to (218.4, 186.4)
- moved R40 175.7 mm to (189.1, 173.1)
- moved U11 175.7 mm to (189.1, 169.0)
- moved C34 175.7 mm to (184.2, 168.3)
- moved C41 175.7 mm to (189.1, 164.9)
- moved C35 175.5 mm to (202.7, 159.0), turned to 90 degrees
- moved U10 174.6 mm to (199.5, 166.1), turned to 0 degrees
- moved R27 172.6 mm to (181.9, 183.9), turned to 0 degrees
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
Commit message: a
Parts:
- moved R6 6.54 mm to (131.3, 105.3), turned to 270 degrees
- moved C8 5.05 mm to (132.5, 101.0)
- moved C6 5.04 mm to (134.4, 101.0)
- moved R1 4.65 mm to (133.9, 104.9), turned to 90 degrees
- moved C1 2.46 mm to (134.2, 109.3), turned to 270 degrees
Routing:
- net GND: track 0.00 -> 13.1 mm
- net N-0000095: track 0.00 -> 13.0 mm
- net N-0000096: track 0.00 -> 5.68 mm
Changed lines of the file:
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@@
   (general
     (links 298)
-    (no_connects 298)
+    (no_connects 291)
     (area 23.132061 56.477 230.100001 190.9832)
     (thickness 1.6)
     (drawings 4)
-    (tracks 0)
+    (tracks 18)
     (zones 0)
     (modules 135)
@@
   )
   (setup
-    (last_trace_width 0.6)
+    (last_trace_width 0.254)
     (user_trace_width 0.4)
     (user_trace_width 0.6)
@@
   )
   (module SM0805 (layer F.Cu)
-    (at 131.75 106 270)
+    (at 132.4991 101.0031 270)
     (attr smd)
     (fp_text reference C8 (at 0 -0.3175 270) (layer F.SilkS)
@@
   )
   (module SM0805 (layer F.Cu)
-    (at 133.75 99.25 180)
+    (at 131.3434 105.3338 270)
     (attr smd)
-    (fp_text reference R6 (at 0 -0.3175 180) (layer F.SilkS)
+    (fp_text reference R6 (at 0 -0.3175 270) (layer F.SilkS)
       (effects (font (size 0.50038 0.50038) (thickness 0.10922)))
     )
-    (fp_text value 100k (at 0 0.381 180) (layer F.SilkS)
+    (fp_text value 100k (at 0 0.381 270) (layer F.SilkS)
       (effects (font (size 0.50038 0.50038) (thickness 0.10922)))
     )
@@
     (fp_line (start 1.524 -0.762) (end 1.524 0.762) (layer F.SilkS) (width 0.09906))
     (fp_line (start 1.524 0.762) (end 0.508 0.762) (layer F.SilkS) (width 0.09906))
-    (pad 1 smd rect (at -0.9525 0 180) (size 0.889 1.397)
+    (pad 1 smd rect (at -0.9525 0 270) (size 0.889 1.397)
       (layers F.Cu F.Paste F.Mask)
       (net 79 N-0000094)
     )
-    (pad 2 smd rect (at 0.9525 0 180) (size 0.889 1.397)
+    (pad 2 smd rect (at 0.9525 0 270) (size 0.889 1.397)
       (layers F.Cu F.Paste F.Mask)
       (net 41 GND)
@@
   )
   (module SM0805 (layer F.Cu)
-    (at 133.75 106 270)
+    (at 134.4168 101.0031 270)
     (attr smd)
     (fp_text reference C6 (at 0 -0.3175 270) (layer F.SilkS)
@@
   )
   (module SM0805 (layer F.Cu)
-    (at 131.75 109.5 90)
+    (at 134.2009 109.2962 270)
     (attr smd)
-    (fp_text reference C1 (at 0 -0.3175 90) (layer F.SilkS)
+    (fp_text reference C1 (at 0 -0.3175 270) (layer F.SilkS)
       (effects (font (size 0.50038 0.50038) (thickness 0.10922)))
     )
-    (fp_text value 100n (at 0 0.381 90) (layer F.SilkS)
+    (fp_text value 100n (at 0 0.381 270) (layer F.SilkS)
       (effects (font (size 0.50038 0.50038) (thickness 0.10922)))
     )
@@
     (fp_line (start 1.524 -0.762) (end 1.524 0.762) (layer F.SilkS) (width 0.09906))
     (fp_line (start 1.524 0.762) (end 0.508 0.762) (layer F.SilkS) (width 0.09906))
-    (pad 1 smd rect (at -0.9525 0 90) (size 0.889 1.397)
+    (pad 1 smd rect (at -0.9525 0 270) (size 0.889 1.397)
       (layers F.Cu F.Paste F.Mask)
       (net 82 N-0000097)
     )
-    (pad 2 smd rect (at 0.9525 0 90) (size 0.889 1.397)
+    (pad 2 smd rect (at 0.9525 0 270) (size 0.889 1.397)
       (layers F.Cu F.Paste F.Mask)
       (net 41 GND)
@@
   )
   (module SM0805 (layer F.Cu)
-    (at 133.75 109.5 270)
+    (at 133.8707 104.8512 90)
     (attr smd)
-    (fp_text reference R1 (at 0 -0.3175 270) (layer F.SilkS)
+    (fp_text reference R1 (at 0 -0.3175 90) (layer F.SilkS)
       (effects (font (size 0.50038 0.50038) (thickness 0.10922)))
     )
-    (fp_text value 10k (at 0 0.381 270) (layer F.SilkS)
+    (fp_text value 10k (at 0 0.381 90) (layer F.SilkS)
       (effects (font (size 0.50038 0.50038) (thickness 0.10922)))
     )
@@
     (fp_line (start 1.524 -0.762) (end 1.524 0.762) (layer F.SilkS) (width 0.09906))
     (fp_line (start 1.524 0.762) (end 0.508 0.762) (layer F.SilkS) (width 0.09906))
-    (pad 1 smd rect (at -0.9525 0 270) (size 0.889 1.397)
+    (pad 1 smd rect (at -0.9525 0 90) (size 0.889 1.397)
       (layers F.Cu F.Paste F.Mask)
       (net 84 VDD)
     )
-    (pad 2 smd rect (at 0.9525 0 270) (size 0.889 1.397)
+    (pad 2 smd rect (at 0.9525 0 90) (size 0.889 1.397)
       (layers F.Cu F.Paste F.Mask)
       (net 82 N-0000097)
@@
   (gr_line (start 230 90) (end 230 190) (angle 90) (layer Dwgs.User) (width 0.2))
   (gr_line (start 130 90) (end 230 90) (angle 90) (layer Dwgs.User) (width 0.2))
+  (segment (start 137.2 93.45) (end 139.75 93.45) (width 0.254) (layer F.Cu) (net 41))
+  (segment (start 134.8 93.45) (end 137.2 93.45) (width 0.254) (layer F.Cu) (net 41))
+  (segment (start 132.25 93.45) (end 134.8 93.45) (width 0.254) (layer F.Cu) (net 41))
+  (segment (start 132.85 97) (end 132.85 94.05) (width 0.254) (layer F.Cu) (net 41))
+  (segment (start 132.85 94.05) (end 132.25 93.45) (width 0.254) (layer F.Cu) (net 41))
+  (segment (start 134.7 97) (end 132.85 97) (width 0.254) (layer F.Cu) (net 41))
+  (segment (start 136 97) (end 136 95.9401) (width 0.254) (layer F.Cu) (net 80))
+  (segment (start 141.0843 98.4758) (end 139.25 100.3101) (width 0.254) (layer F.Cu) (net 80))
+  (segment (start 141.0843 95.9358) (end 141.0843 98.4758) (width 0.254) (layer F.Cu) (net 80))
+  (segment (start 140.4874 95.3389) (end 141.0843 95.9358) (width 0.254) (layer F.Cu) (net 80))
+  (segment (start 136.6012 95.3389) (end 140.4874 95.3389) (width 0.254) (layer F.Cu) (net 80))
+  (segment (start 136 95.9401) (end 136.6012 95.3389) (width 0.254) (layer F.Cu) (net 80))
+  (segment (start 139.25 101.50064) (end 139.25 100.3101) (width 0.254) (layer F.Cu) (net 80))
+  (segment (start 136.65 97) (end 136.65 98.9564) (width 0.254) (layer F.Cu) (net 81))
+  (segment (start 138.3792 100.1522) (end 138.74962 100.52262) (width 0.254) (layer F.Cu) (net 81))
+  (segment (start 137.8458 100.1522) (end 138.3792 100.1522) (width 0.254) (layer F.Cu) (net 81))
+  (segment (start 136.65 98.9564) (end 137.8458 100.1522) (width 0.254) (layer F.Cu) (net 81))
+  (segment (start 138.74962 101.50064) (end 138.74962 100.52262) (width 0.254) (layer F.Cu) (net 81))
 )

Commit message: a
Parts:
- moved R21 10.1 mm to (180.1, 151.9), turned to 270 degrees
- moved R22 9.46 mm to (193.9, 149.4), turned to 270 degrees
- moved R20 7.91 mm to (182.1, 151.9), turned to 270 degrees
- moved R46 4.78 mm to (149.0, 92.3), turned to 90 degrees
- moved R45 4.78 mm to (153.5, 92.3), turned to 90 degrees
- moved R44 4.78 mm to (158.0, 92.3), turned to 90 degrees
- moved D12 4.37 mm to (149.0, 96.8), turned to 90 degrees
- moved D11 4.37 mm to (153.5, 96.8), turned to 90 degrees
- moved D10 4.37 mm to (158.0, 96.8), turned to 90 degrees
- moved C27 2.42 mm to (185.8, 151.1), turned to 270 degrees
- moved R1 0.39 mm to (134.3, 104.9)
- turned C8 to 90 degrees
- turned C6 to 90 degrees
Routing:
- net GND: track 13.1 -> 308.0 mm
- net /v+: track 0.00 -> 111.2 mm
- net /Vin: track 0.00 -> 107.0 mm
- net /v-: track 0.00 -> 105.0 mm
- net VDD: track 0.00 -> 50.4 mm
- net /Eaux-test: track 0.00 -> 45.6 mm
- net /Eaux: track 0.00 -> 34.0 mm
- net /Iref: track 0.00 -> 30.2 mm
- net /servo-vcc: track 0.00 -> 27.2 mm
- net N-0000022: track 0.00 -> 22.5 mm
- net N-0000090: track 0.00 -> 19.2 mm
- net N-00000114: track 0.00 -> 17.9 mm
- net N-00000110: track 0.00 -> 17.7 mm
- net /gate: track 0.00 -> 16.8 mm
- net N-00000117: track 0.00 -> 16.1 mm
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
Commit message: a
Parts:
- added P10, P11, P8, P9: m3-hole, 1pin, F.Cu at (0.00, 0.00)
- moved C4 25.7 mm to (183.7, 120.3)
- moved R4 23.8 mm to (183.7, 125.4)
- moved P2 22.2 mm to (183.7, 122.9), turned to 0 degrees
- moved C21 8.96 mm to (209.1, 106.3)
- moved C22 8.96 mm to (204.3, 125.3)
- moved C24 8.96 mm to (204.3, 132.4)
- moved R14 8.96 mm to (205.8, 112.1)
- moved U8 8.96 mm to (221.4, 106.7)
- moved C19 8.96 mm to (204.5, 104.0)
- moved C28 8.96 mm to (227.1, 110.1)
- moved C31 8.96 mm to (216.8, 108.4)
- moved C32 8.96 mm to (221.1, 122.7)
- moved C36 8.96 mm to (221.6, 129.8)
- moved D3 8.96 mm to (209.9, 114.1)
- moved D5 8.96 mm to (216.5, 115.6)
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Connections:
- MCU1 pad 59: /curr-en -> (no net)
- MCU1 pad 61: /aux-en -> /curr-en
- MCU1 pad 62: (no net) -> /aux-en
Routing:
- net /aux-en: track 0.00 -> 62.7 mm
- net /curr-en: track 0.00 -> 44.1 mm
- net GND: track 308.0 -> 345.2 mm
- net N-00000114: track 0.00 -> 26.4 mm
- net /dac-high: track 0.00 -> 21.7 mm
- net /dac-low: track 0.00 -> 21.4 mm
- net /v-: track 105.0 -> 87.5 mm
- net /Iref-in: track 5.82 -> 21.0 mm
- net /Eref-in: track 0.00 -> 11.7 mm
- net /Eaux-in: track 0.00 -> 11.4 mm
- net /btn-1: track 2.35 -> 9.74 mm
- net /led-0: track 0.00 -> 6.53 mm
- net /btn-2: track 2.35 -> 8.12 mm
- net /Vin: track 107.0 -> 103.2 mm
- net /led-1: track 0.00 -> 3.53 mm
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
Commit message: a
Parts:
- moved P9 292.7 mm to (226.0, 186.0)
- moved P11 244.8 mm to (226.0, 94.0)
- moved P10 229.2 mm to (134.0, 186.0)
- moved P8 163.7 mm to (134.0, 94.0)
- moved R5 5.31 mm to (154.9, 107.0), turned to 180 degrees
- moved C6 4.77 mm to (137.6, 99.9), turned to 180 degrees
- moved C8 2.81 mm to (137.6, 101.8), turned to 180 degrees
- moved R41 1.95 mm to (172.8, 113.6), turned to 0 degrees
- moved C1 1.51 mm to (141.0, 110.4)
- moved R6 1.37 mm to (137.8, 105.3)
- moved P6 0.49 mm to (203.9, 186.0)
- moved P7 0.44 mm to (212.1, 186.0)
- moved P5 0.44 mm to (220.3, 186.0)
Connections:
- MCU1 pad 2: (no net) -> /volt-en
- MCU1 pad 25: (no net) -> /led-0
- MCU1 pad 26: /led-0 -> /led-1
- MCU1 pad 27: /led-1 -> /led-2
- MCU1 pad 29: /led-2 -> /btn-2
- MCU1 pad 33: /btn-2 -> (no net)
- MCU1 pad 58: /volt-en -> (no net)
Routing:
- net GND: track 345.2 -> 565.4 mm
- net /servo-en-400mA: track 0.00 -> 26.8 mm
- net /servo-en-60mA: track 0.00 -> 26.8 mm
- net /suspend: track 5.61 -> 28.2 mm
- net /btn-2: track 8.12 -> 29.2 mm
- net /led-0: track 6.53 -> 24.5 mm
- net /led-2: track 2.55 -> 20.4 mm
- net /src: track 5.42 -> 23.2 mm, vias 0 -> 1
- net /led-1: track 3.53 -> 20.9 mm
- net VDD: track 52.9 -> 63.8 mm, vias 0 -> 1
- net /txd: track 0.00 -> 8.51 mm, vias 0 -> 1
- net /v-: track 87.5 -> 95.8 mm
- net /rxd: track 0.00 -> 8.30 mm, vias 0 -> 1
- net N-0000019: track 4.74 -> 12.2 mm
- net /btn-1: track 9.74 -> 16.7 mm, vias 0 -> 2
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
Commit message: a
Parts:
- moved R36 1.89 mm to (182.4, 114.0), turned to 0 degrees
- moved R31 1.89 mm to (190.7, 114.3), turned to 0 degrees
- moved R37 1.05 mm to (184.3, 109.1)
- moved C40 0.75 mm to (171.3, 110.5)
- moved C33 0.69 mm to (181.1, 110.9)
- moved R42 0.60 mm to (174.8, 109.2)
- moved C5 0.20 mm to (167.8, 120.2), turned to 180 degrees
Routing:
- net /Eref-test: track 5.71 -> 94.1 mm, vias 0 -> 2
- net /v+: track 111.2 -> 152.7 mm, vias 0 -> 1
- net /AVdd: track 7.48 -> 48.6 mm
- net /Eaux-test: track 45.6 -> 75.8 mm
- net GND: track 565.4 -> 594.0 mm
- net /Eaux-in: track 11.4 -> 37.4 mm
- net /rxd: track 8.30 -> 28.7 mm, vias 1 -> 2
- net /Eref-in: track 11.7 -> 31.2 mm
- net N-0000090: track 13.1 -> 27.2 mm
- net /btn-1: track 16.7 -> 27.6 mm
- net /Vbus: track 3.87 -> 13.1 mm, vias 1 -> 2
- net /Iref-in: track 14.1 -> 22.5 mm
- net /txd: track 8.51 -> 13.8 mm, vias 1 -> 2

Commit message: a
Routing:
- net VDD: track 63.8 -> 153.8 mm, vias 1 -> 7
- net GND: track 594.0 -> 668.7 mm, vias 0 -> 1
- net /txd: track 13.8 -> 32.9 mm
- net /dac-high: track 22.8 -> 23.9 mm, vias 0 -> 1
- net /dac-low: track 23.7 -> 24.0 mm, vias 0 -> 1
