File: electrics/scheme/voltamper.kicad_pcb (KiCad board)
At the start: 2 copper layers, 87 x 64 mm, 149 parts, among them K1 swd, K2 servo-1, K3 servo-2, P1 boot, P10 m3-hole, P11 m3-hole, P12 CONN_13X2, P2 boot, P3 -, P4 +, P5 work, P6 aux, P7 ref, P8 m3-hole, P9 m3-hole, Q1 bc857, Q2 bc847, Q3 bc857, Q4 bc847, Q5 irlml2244, Q8 bc847, Q9 bc847, SW1 btn-1, SW2 btn-2, U1 CRYSTAL-4PIN, U10 ADA4000, U11 INA126, U12 SPARTAN-SIP-9007, U13 OPA551, U14 AD825, U15 SPARTAN-SIP-9007, U2 CP2102, U3 MICRO-USB-B, U4 MCP1703T-3302E/CB, U5 MCP1703T-3302E/CB, U6 NCP3063, U8 NCP3063

Commit message: a
Routing:
- net /v-: track 145.7 -> 152.2 mm, vias 4 -> 5
- net N-0000075: track 35.4 -> 33.2 mm
- net /eref-volt: track 67.9 -> 68.9 mm
- added copper zone on F.Cu, net /v-
Changed lines of the file:
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@@
 (kicad_pcb (version 3) (host pcbnew "(2013-07-07 BZR 4022)-stable")
   (general
-    (links 332)
+    (links 333)
     (no_connects 0)
-    (area 129.691889 89.051 217.308111 154.100001)
+    (area 129.691889 89.051 235.5 165.7)
     (thickness 1.6)
     (drawings 17)
-    (tracks 1585)
+    (tracks 1596)
     (zones 0)
     (modules 149)
@@
   (layers
     (15 F.Cu signal)
-    (0 B.Cu signal)
+    (0 B.Cu signal hide)
     (16 B.Adhes user)
     (17 F.Adhes user)
@@
   )
   (setup
-    (last_trace_width 0.6)
+    (last_trace_width 0.4)
     (user_trace_width 0.4)
     (user_trace_width 0.6)
@@
     (mod_text_size 1 1)
     (mod_text_width 0.15)
-    (pad_size 0.9 3)
+    (pad_size 10.41 6.9)
     (pad_drill 0)
     (pad_to_mask_clearance 0)
@@
     )
   )
-  (module OPA551 (layer F.Cu)
-    (at 206.2 124.6)
-    (fp_text reference U13 (at 0 -9.9) (layer F.SilkS)
-      (effects (font (size 1 1) (thickness 0.15)))
-    )
-    (fp_text value OPA551 (at 6.7 -5.4 90) (layer F.SilkS)
-      (effects (font (size 1 1) (thickness 0.15)))
-    )
-    (pad 1 smd rect (at -3.81 3.74) (size 0.9 3)
-      (layers F.Cu F.Paste F.Mask)
-      (net 76 N-0000065)
-    )
-    (pad 2 smd rect (at -2.54 3.74) (size 0.9 3)
-      (layers F.Cu F.Paste F.Mask)
-      (net 78 N-0000071)
-    )
-    (pad 3 smd rect (at -1.27 3.74) (size 0.9 3)
-      (layers F.Cu F.Paste F.Mask)
-    )
-    (pad 4 smd rect (at 0 3.74) (size 0.9 3)
-      (layers F.Cu F.Paste F.Mask)
-      (net 47 /v-)
-    )
-    (pad 5 smd rect (at 1.27 3.74) (size 0.9 3)
-      (layers F.Cu F.Paste F.Mask)
-      (net 46 /v+)
-    )
-    (pad 6 smd rect (at 2.54 3.74) (size 0.9 3)
-      (layers F.Cu F.Paste F.Mask)
-      (net 17 /eaux-volt)
-    )
-    (pad 7 smd rect (at 3.81 3.74) (size 0.9 3)
-      (layers F.Cu F.Paste F.Mask)
-    )
-    (pad 8 smd rect (at 0 -5.51) (size 10.41 6.9)
-      (layers F.Cu F.Paste F.Mask)
-    )
-  )
   (module SPARTAN-SIP-9007 (layer F.Cu)
     (at 194 143.7 180)
@@
     )
   )
+  (module OPA551 (layer F.Cu)
+    (at 206.2 124.6)
+    (fp_text reference U13 (at 0 -9.9) (layer F.SilkS)
+      (effects (font (size 1 1) (thickness 0.15)))
+    )
+    (fp_text value OPA551 (at 0 6.4) (layer F.SilkS)
+      (effects (font (size 1 1) (thickness 0.15)))
+    )
+    (pad 1 smd rect (at -3.81 3.74) (size 0.9 3)
+      (layers F.Cu F.Paste F.Mask)
+      (net 76 N-0000065)
+    )
+    (pad 2 smd rect (at -2.54 3.74) (size 0.9 3)
+      (layers F.Cu F.Paste F.Mask)
+      (net 78 N-0000071)
+    )
+    (pad 3 smd rect (at -1.27 3.74) (size 0.9 3)
+      (layers F.Cu F.Paste F.Mask)
+    )
+    (pad 4 smd rect (at 0 3.74) (size 0.9 3)
+      (layers F.Cu F.Paste F.Mask)
+      (net 47 /v-)
+    )
+    (pad 5 smd rect (at 1.27 3.74) (size 0.9 3)
+      (layers F.Cu F.Paste F.Mask)
+      (net 46 /v+)
+    )
+    (pad 6 smd rect (at 2.54 3.74) (size 0.9 3)
+      (layers F.Cu F.Paste F.Mask)
+      (net 17 /eaux-volt)
+    )
+    (pad 7 smd rect (at 3.81 3.74) (size 0.9 3)
+      (layers F.Cu F.Paste F.Mask)
+    )
+    (pad 4 smd rect (at 0 -5.51) (size 10.41 6.9)
+      (layers F.Cu F.Paste F.Mask)
+      (net 47 /v-)
+    )
+  )
   (dimension 64 (width 0.3) (layer Dwgs.User)
     (gr_text "64.000 mm" (at 228.85 122 90) (layer Dwgs.User)
@@
   (segment (start 188.35 130.05) (end 188.35 132.3) (width 0.4) (layer F.Cu) (net 17))
   (segment (start 184.5025 126.2025) (end 188.35 130.05) (width 0.4) (layer F.Cu) (net 17))
-  (segment (start 187.25 107.65) (end 187.4 107.65) (width 0.4) (layer F.Cu) (net 18))
-  (segment (start 198.6 119.4) (end 199.3 120.1) (width 0.4) (layer F.Cu) (net 18))
-  (segment (start 198.6 118.85) (end 198.6 119.4) (width 0.4) (layer F.Cu) (net 18))
-  (segment (start 187.4 107.65) (end 198.6 118.85) (width 0.4) (layer F.Cu) (net 18))
+  (segment (start 199.45 123) (end 199.45 122.7) (width 0.4) (layer F.Cu) (net 18))
+  (segment (start 185.15 107.65) (end 183.9025 107.65) (width 0.4) (layer F.Cu) (net 18) (status 800000))
+  (segment (start 186.25 108.75) (end 185.15 107.65) (width 0.4) (layer F.Cu) (net 18))
+  (segment (start 187.25 108.75) (end 186.25 108.75) (width 0.4) (layer F.Cu) (net 18))
+  (segment (start 195.75 117.25) (end 187.25 108.75) (width 0.4) (layer F.Cu) (net 18))
+  (segment (start 195.75 120.5) (end 195.75 117.25) (width 0.4) (layer F.Cu) (net 18))
+  (segment (start 197 121.75) (end 195.75 120.5) (width 0.4) (layer F.Cu) (net 18))
+  (segment (start 198.5 121.75) (end 197 121.75) (width 0.4) (layer F.Cu) (net 18))
+  (segment (start 199.45 122.7) (end 198.5 121.75) (width 0.4) (layer F.Cu) (net 18))
+  (segment (start 202.15 124.65) (end 200.7 124.65) (width 0.4) (layer F.Cu) (net 18))
+  (segment (start 199.45 123.4) (end 199.45 123) (width 0.4) (layer F.Cu) (net 18))
+  (segment (start 200.7 124.65) (end 199.45 123.4) (width 0.4) (layer F.Cu) (net 18))
   (segment (start 211.567 140.235) (end 212.965 140.235) (width 0.4) (layer F.Cu) (net 18))
   (segment (start 212.965 140.235) (end 213.35 139.85) (width 0.4) (layer F.Cu) (net 18))
@@
   (segment (start 213.35 128.25) (end 209.75 124.65) (width 0.4) (layer F.Cu) (net 18))
   (segment (start 209.75 124.65) (end 202.15 124.65) (width 0.4) (layer F.Cu) (net 18))
-  (segment (start 202.15 124.65) (end 199.3 121.8) (width 0.4) (layer F.Cu) (net 18))
-  (segment (start 199.3 121.8) (end 199.3 120.1) (width 0.4) (layer F.Cu) (net 18))
-  (segment (start 187.25 107.65) (end 183.9025 107.65) (width 0.4) (layer F.Cu) (net 18))
   (segment (start 203.1 138.9525) (end 201.2 138.9525) (width 0.6) (layer F.Cu) (net 18))
   (segment (start 206.233 138.965) (end 203.1125 138.965) (width 0.6) (layer F.Cu) (net 18))
@@
   (segment (start 195.2393 95.8864) (end 195.2393 97.4612) (width 0.6) (layer F.Cu) (net 46))
   (segment (start 195.2393 97.4612) (end 195.3536 97.5755) (width 0.6) (layer F.Cu) (net 46))
+  (segment (start 206.2 119.09) (end 206.2 114.85) (width 0.6) (layer F.Cu) (net 47) (status 400000))
+  (segment (start 206.175 114.825) (end 204.025 114.825) (width 0.6) (layer B.Cu) (net 47))
+  (segment (start 206.2 114.85) (end 206.175 114.825) (width 0.6) (layer B.Cu) (net 47))
+  (via (at 206.2 114.85) (size 0.889) (layers F.Cu B.Cu) (net 47))
   (segment (start 205.925 116.725) (end 206.15 116.95) (width 0.6) (layer B.Cu) (net 47))
   (segment (start 206.15 135) (end 207 135.85) (width 0.6) (layer B.Cu) (net 47))
@@
   (segment (start 205.925 116.725) (end 204.7 115.5) (width 0.6) (layer B.Cu) (net 47))
   (segment (start 200.45 111.25) (end 198.96 111.25) (width 0.6) (layer B.Cu) (net 47))
-  (segment (start 204.7 115.5) (end 200.45 111.25) (width 0.6) (layer B.Cu) (net 47))
+  (segment (start 204.7 115.5) (end 204.025 114.825) (width 0.6) (layer B.Cu) (net 47))
+  (segment (start 204.025 114.825) (end 200.45 111.25) (width 0.6) (layer B.Cu) (net 47))
   (segment (start 205.9 131.3475) (end 204.4975 131.3475) (width 0.6) (layer F.Cu) (net 47))
   (segment (start 202.55 115.2) (end 198.78 111.43) (width 0.6) (layer B.Cu) (net 47))
@@
   (segment (start 201.2 134.9475) (end 201.4475 134.7) (width 0.6) (layer F.Cu) (net 78))
   (segment (start 201.2 134.9475) (end 201.4475 134.7) (width 0.4) (layer F.Cu) (net 78))
+  (segment (start 194.07 122.0475) (end 194.07 121.93) (width 0.4) (layer F.Cu) (net 79) (status C00000))
+  (segment (start 193.1 116.25) (end 187.975 111.125) (width 0.4) (layer F.Cu) (net 79))
+  (segment (start 193.25 116.25) (end 193.1 116.25) (width 0.4) (layer F.Cu) (net 79))
+  (segment (start 194.5 117.5) (end 193.25 116.25) (width 0.4) (layer F.Cu) (net 79))
+  (segment (start 194.5 121.5) (end 194.5 117.5) (width 0.4) (layer F.Cu) (net 79))
+  (segment (start 194.07 121.93) (end 194.5 121.5) (width 0.4) (layer F.Cu) (net 79) (status 400000))
   (segment (start 171.9025 108) (end 184.7 108) (width 0.4) (layer B.Cu) (net 79))
-  (segment (start 187.975 111.125) (end 189.075 111.125) (width 0.4) (layer F.Cu) (net 79))
   (segment (start 186.7 109.85) (end 187.975 111.125) (width 0.4) (layer F.Cu) (net 79))
   (via (at 186.7 109.85) (size 0.889) (layers F.Cu B.Cu) (net 79))
   (segment (start 186.55 109.85) (end 186.7 109.85) (width 0.4) (layer B.Cu) (net 79))
   (segment (start 184.7 108) (end 186.55 109.85) (width 0.4) (layer B.Cu) (net 79))
-  (segment (start 194.07 122.0475) (end 194.6525 122.0475) (width 0.4) (layer F.Cu) (net 79))
-  (segment (start 194.6525 122.0475) (end 196.1 120.6) (width 0.4) (layer F.Cu) (net 79))
-  (segment (start 196.1 120.6) (end 196.1 118.15) (width 0.4) (layer F.Cu) (net 79))
-  (segment (start 196.1 118.15) (end 189.075 111.125) (width 0.4) (layer F.Cu) (net 79))
   (segment (start 171.9025 108.95) (end 171.9025 108) (width 0.4) (layer B.Cu) (net 79))
   (segment (start 171.9025 108) (end 171.9025 107.05) (width 0.4) (layer B.Cu) (net 79))
@@
       )
     )
+    (polygon
+      (pts        (xy 213.5 124.5) (xy 213.5 112.25) (xy 194.5 110.75) (xy 199 124.5)
+      )
+    )
   )
   (zone (net 49) (net_name GNDA) (layer B.Cu) (hatch edge 0.508)
@@
       )
     )
+  )
+  (zone (net 47) (net_name /v-) (layer F.Cu) (hatch edge 0.508)
+    (connect_pads yes (clearance 0.5))
+    (min_thickness 0.254)
+    (fill (arc_segments 16) (thermal_gap 0.254) (thermal_bridge_width 0.508))
+    (polygon
+      (pts
+        (xy 212.75 123.75) (xy 199.75 123.75) (xy 195.5 111.5) (xy 212.75 113)
+      )
+    )
