File: electrics/scheme-save/voltamper.sch (KiCad schematic (older format))
At the start: 166 parts, among them K1 swd, K2 servo-1, K3 servo-2, P1 boot, P10 m3-hole, P11 m3-hole, P12 CONN_13X2, P2 boot, P3 -, P4 +, P5 work, P6 aux, P7 ref, P8 m3-hole, P9 m3-hole, Q1 bc857, Q2 bc847, Q3 bc857, Q4 bc847, Q5 irlml2244, Q6 bc847, Q7 bc847, Q8 bc847, SW1 btn-1, SW2 btn-2, U1 CRYSTAL-4PIN, U11 INA126, U12 SPARTAN-SIP-9007, U2 CP2102, U3 MICRO-USB-B, U4 MCP1703T-3302E/CB, U5 MCP1703T-3302E/CB, U6 NCP3063, U7 SPARTAN-SIP-9007, U8 NCP3063, U9 SPARTAN-SIP-9007

Commit message: Started changing scheme.
Parts:
- removed C? (x10): 4u7, ~, symbol C
- removed C? (x4): 10n, ~, symbol C
- removed R? (x7): 10k 0.1%, ~, symbol R
- removed R?: 13.3k 0.1%, ~, symbol R
- removed R?: 40k 0.1%, ~, symbol R
- removed R? (x2): 1k 0.1%, ~, symbol R
- removed R? (x8): 16, ~, symbol R
- removed R?: 10, ~, symbol R
- removed U? (x4): AD825, ~, symbol AD825
- removed U?: OPA551, ~, symbol OPA551
- added C20, C26, C27, C35, C37, C39, C42: 100n, ~, symbol C
- added C23, C25, C30: 10n, ~, symbol C
- added C38: 1u, ~, symbol C
- added D4, D6: lm258a, symbol AD8607
- added R17, R18: 10k, ~, symbol R
- added R22, R30, R35: 1k, ~, symbol R
- added R25: 6k8, ~, symbol R
- added U10: TDA2030A, ~, symbol TDA2030A
- R20: value 1k -> 10
Connections:
- net labels added: Eaux, Eaux-test, Eref-test, Vpp/2
- net labels removed: eaux-volt, eref-volt, intermediate, pre-eaux
- wire segments 515 -> 478
- no-connect marks 26 -> 25
Other:
- note added: "-11.7..+11.7"
- note added: "Here opamps in 1:1 mode because later voltage \nis mixed using resistor voltage divider. And \nbecause of this it needs isolation."
- note added: "I +/-50mA => +/-0.5V (G=10) =>+/-5V"
- note added: "This resistor protects two (voltage and current) \ninputs from short circuit when both relays are on."
- note added: "V = +/-10V"
- note added: "Vin=0..3V => Vout=-11.7V..11.7V"
- note removed: "-Vdd*4...+Vdd*4"
- note removed: "Resistorsin different packages."
- moved on the sheet: C34, C41, D7, D8, D9, K2, K3, P5, P6, P7, Q1, Q2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
