File: drawings/chassis/electric/scheme/cam-chassis.sch (KiCad schematic (older format))
At the start: 36 parts

Commit message: a
Parts:
- removed R? (x2): 30k, ~, symbol R
- removed R?: 0, ~, symbol R
- added C?: 1000u, ~, symbol CP1
- added D?: dbg-led, ~, symbol LED
- added D? (x3): light-led, ~, symbol LED
- added Q?: irlml2244, ~, symbol MOSFET_P
- added Q?: NPN, ~, symbol NPN
- added R? (x3): 1k, ~, symbol R
- added R? (x3): 33, ~, symbol R
- added R?: 30k, ~, symbol R
Connections:
- wire segments 124 -> 137

Commit message: a
Parts:
- removed U?: CRYSTAL-4PIN, ~, symbol CRYSTAL-4PIN
- added K1: pyro, Pin_Headers:Pin_Header_Straight_1x03, symbol CONN_3
- added P1, P2, P3, P4, P5, P6: TST, Pin_Headers:Pin_Header_Straight_1x01, symbol TST
- added U1: crystal-4pin, crystal-smd-5x3:CRYSTAL-SMD-5x3, symbol crystal-4pin
- C1, C2, C3, C4, C5, C6, C8: renamed from C?; footprint ~ -> Capacitors_SMD:C_0805
- C7: renamed from C?; footprint ~ -> Discret:C2V10
- D1, D4, D5, D6: renamed from D?; footprint ~ -> LEDs:LED-5MM
- D2, D3: renamed from D?; footprint ~ -> MY_STAB-5-mm
- IC1: renamed from IC?; footprint TQFP32 -> Housings_QFP:TQFP-32_7x7mm_Pitch0.8mm
- P7: renamed from P?; value CONN_3X2 -> servo; footprint (none) -> Pin_Headers:Pin_Header_Straight_2x03
- Q1, Q2, Q3, Q4, Q5, Q6, Q7: renamed from Q?; footprint ~ -> Housings_SOT-23_SOT-143_TSOT-6:SOT-23
- R1, R10, R11, R12, R13, R14, R15, R16, R17, R18, R19, R2, R20, R21, R22, R3, R4, R5, R6, R7, R8, R9: renamed from R?; footprint ~ -> Resistors_SMD:R_0805
- U2: renamed from U?; footprint ~ -> micro-usb-b:micro-usb-b
Connections:
- net labels added: dbg-led, led, mcu-vcc, pyro-sen
- net labels removed: avcc, vcc1, vcc2
- wire segments 137 -> 161
- no-connect marks 2 -> 10
Other:
- moved on the sheet: C6, D1, R9

Commit message: a
Parts:
- removed Q1: bc857, Housings_SOT-23_SOT-143_TSOT-6:SOT-23, symbol PNP
- removed Q2: bc847, Housings_SOT-23_SOT-143_TSOT-6:SOT-23, symbol NPN
- removed R1: 10, Resistors_SMD:R_0805, symbol R
- removed R14: 100k, Resistors_SMD:R_0805, symbol R
- removed R2: 1k, Resistors_SMD:R_0805, symbol R
- removed R4: 30k, Resistors_SMD:R_0805, symbol R
- D2, D3: footprint MY_STAB-5-mm -> my_foots:MY_STAB-3.5-mm
- Q5, Q7: footprint Housings_SOT-23_SOT-143_TSOT-6:SOT-23 -> libs:SOT23GDS
Connections:
- net labels added: servo-vcc
- net labels removed: servo-en-60mA, vcc
- wire segments 161 -> 145
- no-connect marks 10 -> 11
Other:
- moved on the sheet: C2, C7, Q3, Q4, Q5, R5, R6, R7, R8

Commit message: a
Changed lines of the file:
@@
 Text Label 8250 900  0    60   ~ 0
 gnd
-Text Label 7350 1100 0    60   ~ 0
+Text Label 10400 1100 0    60   ~ 0
 servo1
 Text Label 9450 900  0    60   ~ 0
 gnd
-Text Label 10350 1100 0    60   ~ 0
+Text Label 7350 1100 0    60   ~ 0
 servo2
 $Comp
