File: drawings/chassis/electric/scheme/cam-chassis.kicad_pcb (KiCad board)
At the start: 2 copper layers, 54 parts, among them IC1 ATMEGA8-AI, K1 pyro, P1 TST, P2 TST, P3 TST, P4 TST, P5 TST, P6 TST, P7 servo, Q1 bc857, Q2 bc847, Q3 bc857, Q4 bc847, Q5 irlml2244, Q6 NPN, Q7 irlml2244, U1 CRYSTAL-4PIN, U2 MICRO-USB-B

Commit message: a
Parts:
- moved R16 68.8 mm to (190.7, 115.8), turned to 270 degrees
- moved C8 65.9 mm to (193.3, 109.2), turned to 180 degrees
- moved R13 63.2 mm to (187.3, 115.8), turned to 90 degrees
- moved R12 62.3 mm to (189.0, 115.8), turned to 90 degrees
- moved D2 61.8 mm to (192.2, 112.6), turned to 180 degrees
- moved D3 41.4 mm to (184.2, 112.6)

Commit message: a
Parts:
- removed Q1: bc857, Housings_SOT-23_SOT-143_TSOT-6:SOT-23
- removed Q2: bc847, Housings_SOT-23_SOT-143_TSOT-6:SOT-23
- removed R1: 10, Resistors_SMD:R_0805
- removed R14: 100k, Resistors_SMD:R_0805
- removed R2: 1k, Resistors_SMD:R_0805
- removed R4: 30k, Resistors_SMD:R_0805
- D2, D3: footprint my_foots:MY_STAB-5-mm -> my_foots:MY_STAB-3.5-mm
- Q5, Q7: footprint Housings_SOT-23_SOT-143_TSOT-6:SOT-23 -> libs:SOT23GDS
- U1: value CRYSTAL-4PIN -> crystal-4pin
- moved C1 91.3 mm to (116.0, 92.7), turned to 180 degrees
- moved U1 85.2 mm to (115.9, 96.6), turned to 270 degrees
- moved D2 84.0 mm to (111.0, 91.0)
- moved R13 82.7 mm to (107.5, 94.0)
- moved R12 82.7 mm to (109.2, 94.0)
- moved R16 82.6 mm to (111.0, 94.0)
- moved IC1 82.2 mm to (108.3, 102.4), turned to 180 degrees
- moved U2 82.1 mm to (108.0, 85.5)
- moved C8 82.0 mm to (114.1, 88.1), turned to 270 degrees
- moved D3 81.4 mm to (105.8, 91.0)
- moved C2 77.7 mm to (118.8, 97.3), turned to 90 degrees
- moved Q4 61.2 mm to (101.5, 107.6), turned to 180 degrees
- moved P6 58.6 mm to (99.7, 85.2)
- moved C6 50.4 mm to (102.0, 102.5), turned to 90 degrees
- moved P4 50.3 mm to (99.7, 89.8)
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Connections:
- C7 pad 1: VCC -> /servo-vcc
- IC1 pad 10: N-0000025 -> (no net)
- IC1 pad 11: N-0000024 -> (no net)
- IC1 pad 12: /d+ -> /d-
- IC1 pad 13: /d- -> /d+
- IC1 pad 14: N-0000023 -> (no net)
- IC1 pad 19: N-0000029 -> (no net)
- IC1 pad 22: N-0000028 -> (no net)
- IC1 pad 23: /servo-en-60mA -> (no net)
- IC1 pad 25: N-0000030 -> (no net)
- IC1 pad 30: N-0000021 -> (no net)
- IC1 pad 31: /usb-en -> (no net)
- IC1 pad 9: N-0000026 -> /usb-en
- P7 pad 3: VCC -> /servo-vcc
- P7 pad 4: VCC -> /servo-vcc
- Q6 pad 3: N-0000032 -> Net-(Q6-Pad3)
- R17 pad 2: N-0000032 -> Net-(Q6-Pad3)
- R20 pad 1: N-0000033 -> Net-(Q7-PadD)
- R21 pad 1: N-0000033 -> Net-(Q7-PadD)
- R22 pad 1: N-0000033 -> Net-(Q7-PadD)
- U1 pad 1: N-0000038 -> /xtal2
- U1 pad 2: N-0000039 -> (no net)
- U1 pad 3: /xtal2 -> /xtal1
- U1 pad 4: /xtal1 -> (no net)
Routing:
- net GND: track 0.00 -> 45.0 mm
- net VCC: track 0.00 -> 26.7 mm
- net /d-: track 0.00 -> 13.0 mm
- net /xtal2: track 0.00 -> 8.35 mm
- net /xtal1: track 0.00 -> 7.34 mm
- net Net-(D2-Pad2): track 0.00 -> 6.90 mm
- net /src: track 0.00 -> 6.74 mm
- net /led: track 0.00 -> 5.99 mm
- net Net-(R18-Pad1): track 0.00 -> 5.54 mm
- net Net-(D3-Pad2): track 0.00 -> 5.11 mm
- net /d+: track 0.00 -> 3.37 mm
- net /usb-en: track 0.00 -> 3.24 mm
- net /gate: track 0.00 -> 1.61 mm

Commit message: a
Parts:
- moved D4 29.2 mm to (141.0, 104.0)
- moved D5 29.2 mm to (139.5, 95.5)
- moved D6 29.2 mm to (146.5, 99.0)
- moved Q6 29.2 mm to (131.0, 96.0)
- moved Q7 29.2 mm to (132.0, 99.5)
- moved R11 29.2 mm to (128.0, 95.0)
- moved R15 29.2 mm to (131.0, 93.5)
- moved R17 29.2 mm to (129.0, 98.0)
- moved R20 29.2 mm to (136.0, 103.0)
- moved R21 29.2 mm to (134.5, 96.5)
- moved R22 29.2 mm to (144.5, 94.0)
- moved R3 1.17 mm to (110.4, 109.6)
- moved C3 0.98 mm to (113.9, 109.0)
- moved R10 0.40 mm to (127.5, 110.5)
- moved R19 0.40 mm to (130.6, 110.5)
Connections:
- R10 pad 2: /servo1 -> /servo2
- R19 pad 1: /servo2 -> /servo1
Routing:
- net /rst: track 0.00 -> 33.7 mm, vias 0 -> 1
- net /servo1: track 0.00 -> 32.5 mm, vias 0 -> 2
- net /servo2: track 0.00 -> 25.4 mm, vias 0 -> 2
- net /gate: track 1.61 -> 25.3 mm
- net GND: track 45.0 -> 65.1 mm
- net /mosi: track 0.00 -> 17.1 mm
- net VCC: track 26.7 -> 41.9 mm
- net /miso: track 0.00 -> 14.5 mm
- net /sck: track 0.00 -> 12.8 mm
- net /servo-vcc: track 0.00 -> 10.4 mm
- net /pyro-sen: track 0.00 -> 9.59 mm, vias 0 -> 1
- net Net-(P7-Pad5): track 0.00 -> 2.65 mm
- net Net-(P7-Pad6): track 0.00 -> 2.42 mm
- net Net-(D1-Pad1): track 0.00 -> 2.16 mm
- net Net-(Q6-Pad3): track 0.00 -> 2.02 mm
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
Commit message: Done with routing.
Parts:
- moved C7 0.10 mm to (122.9, 89.6)
Routing:
- net GND: track 65.1 -> 256.6 mm, vias 0 -> 3
- net VCC: track 41.9 -> 138.5 mm, vias 0 -> 5
- net /pyro-sen: track 9.59 -> 70.4 mm
- net Net-(Q7-PadD): track 0.00 -> 22.8 mm
- net /servo-vcc: track 10.4 -> 26.2 mm
- net /led: track 5.99 -> 20.8 mm
- net Net-(D6-Pad1): track 0.00 -> 5.09 mm
- net Net-(D5-Pad1): track 0.00 -> 3.75 mm
- net Net-(D4-Pad1): track 0.00 -> 3.75 mm
- net /rst: track 33.7 -> 37.4 mm
- net Net-(Q6-Pad2): track 0.00 -> 2.60 mm
- net Net-(Q6-Pad3): track 2.02 -> 3.64 mm
- added copper zone on B.Cu, net GND
- added copper zone on F.Cu, net GND
Other:
- board outline added: 51.5 x 28.5 mm

Commit message: a
Parts:
- moved K1 2.35 mm to (143.5, 85.5)
Routing:
- net VCC: track 138.5 -> 141.0 mm
- net /pyro-sen: track 70.4 -> 68.5 mm
- net GND: track 256.6 -> 257.3 mm

Commit message: a
Parts:
- moved K1 7.00 mm to (143.5, 92.5)
- moved D5 6.04 mm to (137.0, 101.0)
- moved D4 5.39 mm to (139.0, 109.0)
- moved R20 5.39 mm to (134.0, 108.0)
- moved D6 4.27 mm to (145.0, 103.0)
- moved R22 3.16 mm to (143.5, 97.0)
- moved R21 3.00 mm to (137.5, 96.5), turned to 180 degrees
Routing:
- net GND: track 257.3 -> 239.9 mm
- net /pyro-sen: track 68.5 -> 57.7 mm
- net VCC: track 141.0 -> 135.7 mm
- net Net-(D6-Pad1): track 5.09 -> 6.30 mm
- net Net-(D5-Pad1): track 3.75 -> 4.84 mm
- net Net-(Q7-PadD): track 22.8 -> 21.8 mm
